File: pdn-brain/pdn-brain.kicad_pcb (KiCad board)
At the start: 2 copper layers, 86.4 x 38.1 mm, 16 parts, among them CN1 PH-6AW_C722785, CN2 PH-4AW_C722777, CN3 PH-4AW_C722777, SW4 BOOT, U6 ESP32-S3-WROOM-1(N8R8)

Commit message: 2025 Production Files.
Parts:
- removed C7: 1uF, global:C0805
- added C1: 1uF, global:C0402, F.Cu at (162.1, 55.9)
Connections:
- R12 pad 1: /3.3v -> /+3.3V
