File: pdn-brain/pdn-brain.kicad_sch (KiCad schematic)
At the start: 16 parts, among them CN1 PH-6AW_C722785, CN2 PH-4AW_C722777, CN3 PH-4AW_C722777, SW4 BOOT, U6 ESP32-S3-WROOM-1(N8R8)

Commit message: 2025 Production Files.
Parts:
- removed C7: 1uF, global:C0805, symbol Device:C
- added C1: 1uF, global:C0402, symbol global:CL05A105KO5NNNC
Connections:
- net GND: now also C1.1
- net at R12.2, U6.3 (EN): now also C1.2
Changed lines of the file:
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@@
 	)
 	(symbol
-		(lib_id "Device:C")
-		(at 53.34 71.12 90)
+		(lib_id "global:CL05A105KO5NNNC")
+		(at 53.34 71.12 0)
 		(unit 1)
 		(exclude_from_sim no)
@@
 		(dnp no)
 		(fields_autoplaced yes)
-		(property "Reference" "C7"
-			(at 53.34 64.77 90)
+		(property "Reference" "C1"
+			(at 53.34 64.77 0)
 			(effects
 				(font
@@
 		)
 		(property "Value" "1uF"
-			(at 53.34 67.31 90)
+			(at 53.34 67.31 0)
 			(effects
 				(font
@@
 			)
 		)
-		(property "Footprint" "global:C0805"
-			(at 57.15 70.1548 0)
+		(property "Footprint" "global:C0402"
+			(at 53.34 78.74 0)
 			(effects
 				(font
@@
 			)
 		)
-		(property "Datasheet" "~"
-			(at 53.34 71.12 0)
+		(property "Datasheet" "https://lcsc.com/product-detail/Multilayer-Ceramic-Capacitors-MLCC-SMD-SMT_SAMSUNG_CL05A105KO5NNNC_1uF-105-10-16V_C29266.html"
+			(at 53.34 81.28 0)
 			(effects
 				(font
@@
 			)
 		)
-		(property "LCSC Part" "C2932475"
-			(at 53.34 71.12 0)
+		(property "LCSC Part" "C29266"
+			(at 53.34 83.82 0)
 			(effects
 				(font
@@
 		)
 		(instances
-			(project "pdn-brain"
+			(project ""
 				(path "/df0bc267-025e-4c4e-a09b-51ff87d0c1db"
-					(reference "C7")
+					(reference "C1")
 					(unit 1)
 				)
