File: pdn-power/pdn-power.kicad_pcb (KiCad board)
At the start: 2 copper layers, 48.8 x 25.4 mm, 35 parts, among them CN1 PH-3AW_C722773, CN2 PH-3AW_C722773, CN3 PH-4AW_C722777, J2 GH-2AW R, Q1 FS8205A, SW1 On/Off Switch, U1 TP4056, U2 DW01A, U3 MT3608, U4 LDL1117S33R

Commit message: 2025 Production Files.
Parts:
- added H2: MountingHole, MountingHole:MountingHole_2.2mm_M2_Pad_TopBottom, F.Cu at (139.2, 93.5)
- C6: footprint global:C0805 -> global:C0402
- LED_2: value RED -> GREEN
- moved CN1 1.15 mm to (133.3, 91.6)
- moved CN2 1.15 mm to (145.4, 91.6)
- moved C6 0.36 mm to (141.9, 104.6)
Routing:
- net +3.3V: track 76.0 -> 77.4 mm
- net +5V: track 48.1 -> 49.4 mm
