File: pdn-power/pdn-power.kicad_sch (KiCad schematic)
At the start: 35 parts, among them CN1 PH-3AW_C722773, CN2 PH-3AW_C722773, CN3 PH-4AW_C722777, J2 GH-2AW R, Q1 FS8205A, SW1 On/Off Switch, U1 TP4056, U2 DW01A, U3 MT3608, U4 LDL1117S33R

Commit message: 2025 Production Files.
Parts:
- removed C6: 1uF, global:C0805, symbol Device:C
- added C6: 1uF, global:C0402, symbol global:CL05A105KO5NNNC
- added H2: MountingHole, MountingHole:MountingHole_2.2mm_M2_Pad_TopBottom, symbol Mechanical:MountingHole
- LED_2: value RED -> GREEN; LCSC Part C965799 -> C965804
Connections:
- net GND: now also C6.2
- net VBATT: now also C6.1
Changed lines of the file:
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@@
 	)
 	(junction
-		(at 102.87 163.83)
+		(at 232.41 106.68)
 		(diameter 0)
 		(color 0 0 0 0)
 	)
 	(junction
-		(at 53.34 147.32)
+		(at 102.87 163.83)
 		(diameter 0)
 		(color 0 0 0 0)
 	)
 	(junction
-		(at 171.45 127)
+		(at 53.34 147.32)
 		(diameter 0)
 		(color 0 0 0 0)
 	)
 	(junction
-		(at 232.41 106.68)
+		(at 171.45 127)
 		(diameter 0)
 		(color 0 0 0 0)
@@
 	(wire
 		(pts
+			(xy 232.41 106.68) (xy 232.41 118.11)
+		)
+		(stroke
+			(width 0)
+			(type default)
+		)
+	)
+	(wire
+		(pts
 			(xy 33.02 74.93) (xy 33.02 85.09)
 		)
@@
 	(wire
 		(pts
-			(xy 232.41 106.68) (xy 232.41 118.11)
-		)
-		(stroke
-			(width 0)
-			(type default)
-		)
-	)
-	(wire
-		(pts
 			(xy 45.72 74.93) (xy 53.34 74.93)
 		)
@@
 	)
 	(symbol
-		(lib_id "Device:C")
-		(at 236.22 106.68 90)
+		(lib_id "Mechanical:MountingHole")
+		(at 255.27 123.19 0)
 		(unit 1)
 		(exclude_from_sim no)
@@
 		(on_board yes)
 		(dnp no)
-		(property "Reference" "C6"
-			(at 236.22 100.33 90)
+		(fields_autoplaced yes)
+		(property "Reference" "H2"
+			(at 257.81 122.555 0)
 			(effects
 				(font
 					(size 1.27 1.27)
 				)
+				(justify left)
 			)
 		)
-		(property "Value" "1uF"
-			(at 236.22 102.87 90)
+		(property "Value" "MountingHole"
+			(at 257.81 125.095 0)
 			(effects
 				(font
 					(size 1.27 1.27)
 				)
+				(justify left)
 			)
 		)
-		(property "Footprint" "global:C0805"
-			(at 240.03 105.7148 0)
+		(property "Footprint" "MountingHole:MountingHole_2.2mm_M2_Pad_TopBottom"
+			(at 255.27 123.19 0)
 			(effects
 				(font
@@
 		)
 		(property "Datasheet" "~"
-			(at 236.22 106.68 0)
+			(at 255.27 123.19 0)
 			(effects
 				(font
@@
 		)
 		(property "Description" ""
-			(at 236.22 106.68 0)
+			(at 255.27 123.19 0)
 			(effects
 				(font
@@
 			)
 		)
-		(property "LCSC Part" "C2932475"
-			(at 236.22 106.68 0)
-			(effects
-				(font
-					(size 1.27 1.27)
-				)
-				(hide yes)
-			)
-		)
-		(pin "1"
-		)
-		(pin "2"
-		)
 		(instances
-			(project "pdn-power"
+			(project "power-v2"
 				(path "/df0bc267-025e-4c4e-a09b-51ff87d0c1db"
-					(reference "C6")
+					(reference "H2")
 					(unit 1)
 				)
@@
 			)
 		)
-		(property "Value" "RED"
+		(property "Value" "GREEN"
 			(at 52.07 121.92 90)
 			(effects
@@
 			)
 		)
-		(property "LCSC Part" "C965799"
+		(property "LCSC Part" "C965804"
 			(at 59.69 119.38 0)
 			(effects
@@
 					(unit 1)
 				)
+			)
+		)
+	)
+	(symbol
+		(lib_id "global:CL05A105KO5NNNC")
+		(at 236.22 106.68 0)
+		(unit 1)
+		(exclude_from_sim no)
+		(in_bom yes)
+		(on_board yes)
+		(dnp no)
+		(fields_autoplaced yes)
+		(property "Reference" "C6"
+			(at 236.22 100.33 0)
+			(effects
+				(font
+					(size 1.27 1.27)
+				)
+			)
+		)
+		(property "Value" "1uF"
+			(at 236.22 102.87 0)
+			(effects
+				(font
+					(size 1.27 1.27)
+				)
+			)
+		)
+		(property "Footprint" "global:C0402"
+			(at 236.22 114.3 0)
+			(effects
+				(font
+					(size 1.27 1.27)
+				)
+				(hide yes)
+			)
+		)
+		(property "Datasheet" "https://lcsc.com/product-detail/Multilayer-Ceramic-Capacitors-MLCC-SMD-SMT_SAMSUNG_CL05A105KO5NNNC_1uF-105-10-16V_C29266.html"
+			(at 236.22 116.84 0)
+			(effects
+				(font
+					(size 1.27 1.27)
+				)
+				(hide yes)
+			)
+		)
+		(property "Description" ""
+			(at 236.22 106.68 0)
+			(effects
+				(font
+					(size 1.27 1.27)
+				)
+				(hide yes)
+			)
+		)
+		(property "LCSC Part" "C29266"
+			(at 236.22 119.38 0)
+			(effects
+				(font
+					(size 1.27 1.27)
+				)
+				(hide yes)
+			)
+		)
+		(pin "1"
+		)
+		(pin "2"
+		)
+		(instances
+			(project ""
+				(path "/df0bc267-025e-4c4e-a09b-51ff87d0c1db"
+					(reference "C6")
+					(unit 1)
+				)
