File: pdn-user/pdn-user.kicad_pcb (KiCad board)
At the start: 2 copper layers, 45.7 x 68.6 mm, 26 parts, among them CN1 PH-3AW_C722773, CN2 PH-4AW_C722777, Q2 BJT 2222A, SW1 Primary Button, SW2 Secondary Button

Commit message: 2025 Production Files.
Parts:
- added H1: MountingHole, MountingHole:MountingHole_2.2mm_M2_Pad_TopBottom, F.Cu at (143.2, 113.2)
- added H2: MountingHole, MountingHole:MountingHole_2.2mm_M2_Pad_TopBottom, F.Cu at (166.5, 105.7)
- moved SW2 1.27 mm to (154.6, 102.6)
- moved SW1 1.26 mm to (154.6, 74.6)
Routing:
- net +5V: track 169.1 -> 173.4 mm
- net Net-(R1-Pad2): track 7.71 -> 8.45 mm
- net Net-(R2-Pad1): track 10.7 -> 10.2 mm
- net BT_SEC: track 43.5 -> 43.0 mm
- net BT_PRIM: track 14.7 -> 14.2 mm
