File: pdn-user/pdn-user.kicad_sch (KiCad schematic)
At the start: 26 parts, among them CN1 PH-3AW_C722773, CN2 PH-4AW_C722777, Q2 BJT 2222A, SW1 Primary Button, SW2 Secondary Button

Commit message: 2025 Production Files.
Parts:
- added H1, H2: MountingHole, MountingHole:MountingHole_2.2mm_M2_Pad_TopBottom, symbol Mechanical:MountingHole
Other:
- moved on the sheet: C1, C2, C3, C4, C5, C6, LED1, LED2, LED3, LED4, LED5, LED6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
